Commit message: Update hook model

File: urdf/hook/hook.urdf (robot description, URDF)
Before this commit: robot hook, 1 links, 0 joints
Links:
- link link: geometry collision cylinder length=0.3 radius=0.0025; visual cylinder length=0.3 radius=0.0025

File: urdf/hook/plate_visual.urdf (robot description, URDF)
Before this commit: robot plate, 1 links, 0 joints
Links:
- link link: geometry visual box size=0.01 1.2 1.6
